File: MOSSbp_Sensor_Board/MOSSbp_Sensor_Board.sch (KiCad schematic (older format))
At the start: 6 parts, among them J1 I2C, U1 BME680

Commit message: Finished PCB board
Parts:
- added C3, C4: 100n, Capacitor_SMD:C_0603_1608Metric_Pad1.05x0.95mm_HandSolder, symbol Device:C
- added H1, H2, H3, H4: MH, MountingHole:MountingHole_2.2mm_M2_ISO14580_Pad, symbol Mechanical:MountingHole_Pad
- added U2: BMI160, digikey-footprints:BMI160, symbol dk_Motion-Sensors-IMUs-Inertial-Measurement-Units:BMI160
- C1, C2: footprint (none) -> Capacitor_SMD:C_0603_1608Metric_Pad1.05x0.95mm_HandSolder; Digi-Key_PN (none) -> 311-1341-1-ND
- R1, R2: footprint (none) -> Resistor_SMD:R_0603_1608Metric_Pad1.05x0.95mm_HandSolder; Digi-Key_PN (none) -> 311-4.7KGRCT-ND
Connections:
- net +3V3: now also C3.1, C4.1, U2.12 (CSB), U2.5 (VDDIO), U2.8 (VDD)
- net GND: now also C3.2, C4.2, H1.1, H2.1, H3.1, H4.1, U2.6 (GND), U2.7 (GND)
- net I2C_SCL: now also U2.13 (SC)
- net I2C_SDA: now also U2.14 (SD)
- no-connect marks 0 -> 7
Other:
- moved on the sheet: C1, C2, J1, R1, R2, U1
